File: CH552-USB-Devboard/CH552-USB-Devboard.sch (KiCad schematic (older format))
At the start: 23 parts, among them J1 Conn_01x10_Male, J2 Conn_01x10_Male, J3 USB_A, SW1 SW_Push, SW2 SW_Push, U1 CH552T, U2 CH552G, Y1 Crystal

Commit message: started on layout
Parts:
- removed J3: USB_A, Connector_USB:USB_A_CNCTech_1001-011-01101_Horizontal, symbol Connector:USB_A
- added J3: USB_B_Micro, digikey-footprints:USB_Micro_B_Female_10118193-0001LF, symbol Connector:USB_B_Micro
- SW1, SW2: footprint Button_Switch_SMD:SW_DIP_SPSTx01_Slide_6.7x4.1mm_W6.73mm_P2.54mm_LowProfile_JPin -> Button_Switch_SMD:SW_SPST_PTS810
Changed lines of the file:
@@
 EESchema Schematic File Version 4
+LIBS:CH552-USB-Devboard-cache
 EELAYER 26 0
 EELAYER END
@@
 $EndComp
 $Comp
-L Connector:USB_A J3
-U 1 1 5E91FC86
-P 7750 1350
-F 0 "J3" H 7805 1817 50  0000 C CNN
-F 1 "USB_A" H 7805 1726 50  0000 C CNN
-F 2 "Connector_USB:USB_A_CNCTech_1001-011-01101_Horizontal" H 7900 1300 50  0001 C CNN
-F 3 " ~" H 7900 1300 50  0001 C CNN
-	1    7750 1350
-	1    0    0    -1
-$EndComp
-$Comp
 L Switch:SW_Push SW1
 U 1 1 5E91FDDD
@@
 F 0 "SW1" H 1500 2285 50  0000 C CNN
 F 1 "SW_Push" H 1500 2194 50  0000 C CNN
-F 2 "Button_Switch_SMD:SW_DIP_SPSTx01_Slide_6.7x4.1mm_W6.73mm_P2.54mm_LowProfile_JPin" H 1500 2200 50  0001 C CNN
+F 2 "Button_Switch_SMD:SW_SPST_PTS810" H 1500 2200 50  0001 C CNN
 F 3 "" H 1500 2200 50  0001 C CNN
 	1    1500 2000
@@
 F 0 "SW2" V 4096 2002 50  0000 R CNN
 F 1 "SW_Push" V 4005 2002 50  0000 R CNN
-F 2 "Button_Switch_SMD:SW_DIP_SPSTx01_Slide_6.7x4.1mm_W6.73mm_P2.54mm_LowProfile_JPin" H 4050 2250 50  0001 C CNN
+F 2 "Button_Switch_SMD:SW_SPST_PTS810" H 4050 2250 50  0001 C CNN
 F 3 "" H 4050 2250 50  0001 C CNN
 	1    4050 2050
@@
 Wire Wire Line
 	3100 3200 3100 3400
+$Comp
+L Connector:USB_B_Micro J3
+U 1 1 5E92FB1C
+P 7750 1350
+F 0 "J3" H 7805 1817 50  0000 C CNN
+F 1 "USB_B_Micro" H 7805 1726 50  0000 C CNN
+F 2 "digikey-footprints:USB_Micro_B_Female_10118193-0001LF" H 7900 1300 50  0001 C CNN
+F 3 "~" H 7900 1300 50  0001 C CNN
+	1    7750 1350
+	1    0    0    -1
+$EndComp
 $EndSCHEMATC

Commit message: first route done
Connections:
- wire segments 118 -> 119
Changed lines of the file:
@@
 Wire Wire Line
 	10150 1500 10350 1500
-Wire Wire Line
-	10550 1500 10800 1500
 $Comp
 L Device:R_Small R5
@@
 	10550 1800 10800 1800
 Wire Wire Line
-	10800 1150 10800 1800
+	10800 1150 10800 1500
 Wire Wire Line
 	9850 1800 9550 1800
@@
 	1    0    0    -1
 $EndComp
+Wire Wire Line
+	10550 1500 10800 1500
+Connection ~ 10800 1500
+Wire Wire Line
+	10800 1500 10800 1800
+$Comp
+L power:VCC #PWR?
+U 1 1 5EA08550
+P 10800 800
+F 0 "#PWR?" H 10800 650 50  0001 C CNN
+F 1 "VCC" H 10817 973 50  0000 C CNN
+F 2 "" H 10800 800 50  0001 C CNN
+F 3 "" H 10800 800 50  0001 C CNN
+	1    10800 800
+	1    0    0    -1
+$EndComp

Commit message: ROUTING COMPLETE AND DRC DONE READY FOR SILK
Changed lines of the file:
@@
 L Device:R_Small R3
 U 1 1 5E91F991
-P 10450 1150
-F 0 "R3" V 10254 1150 50  0000 C CNN
-F 1 "330r" V 10345 1150 50  0000 C CNN
-F 2 "Resistor_SMD:R_0603_1608Metric_Pad1.05x0.95mm_HandSolder" H 10450 1150 50  0001 C CNN
-F 3 "~" H 10450 1150 50  0001 C CNN
-	1    10450 1150
+P 10500 1800
+F 0 "R3" V 10304 1800 50  0000 C CNN
+F 1 "330r" V 10395 1800 50  0000 C CNN
+F 2 "Resistor_SMD:R_0603_1608Metric_Pad1.05x0.95mm_HandSolder" H 10500 1800 50  0001 C CNN
+F 3 "~" H 10500 1800 50  0001 C CNN
+	1    10500 1800
 	0    1    1    0
 $EndComp
@@
 L Device:LED D1
 U 1 1 5E91FEF9
-P 10000 1150
-F 0 "D1" H 9991 1366 50  0000 C CNN
-F 1 "LED" H 9991 1275 50  0000 C CNN
-F 2 "LEDs:LED_0805" H 10000 1150 50  0001 C CNN
-F 3 "~" H 10000 1150 50  0001 C CNN
-	1    10000 1150
-	1    0    0    -1
-$EndComp
-Wire Wire Line
-	10150 1150 10350 1150
-Wire Wire Line
-	10550 1150 10800 1150
-Wire Wire Line
-	10800 1150 10800 800
+P 10050 1800
+F 0 "D1" H 10041 2016 50  0000 C CNN
+F 1 "LED" H 10041 1925 50  0000 C CNN
+F 2 "LEDs:LED_0805" H 10050 1800 50  0001 C CNN
+F 3 "~" H 10050 1800 50  0001 C CNN
+	1    10050 1800
+	-1   0    0    1
+$EndComp
+Wire Wire Line
+	10200 1800 10400 1800
+Wire Wire Line
+	10600 1800 10850 1800
 $Comp
 L Device:R_Small R4
 U 1 1 5E9203E3
-P 10450 1500
-F 0 "R4" V 10254 1500 50  0000 C CNN
-F 1 "330r" V 10345 1500 50  0000 C CNN
-F 2 "Resistor_SMD:R_0603_1608Metric_Pad1.05x0.95mm_HandSolder" H 10450 1500 50  0001 C CNN
-F 3 "~" H 10450 1500 50  0001 C CNN
-	1    10450 1500
+P 10500 2150
+F 0 "R4" V 10304 2150 50  0000 C CNN
+F 1 "330r" V 10395 2150 50  0000 C CNN
+F 2 "Resistor_SMD:R_0603_1608Metric_Pad1.05x0.95mm_HandSolder" H 10500 2150 50  0001 C CNN
+F 3 "~" H 10500 2150 50  0001 C CNN
+	1    10500 2150
 	0    1    1    0
 $EndComp
@@
 L Device:LED D2
 U 1 1 5E9203EA
-P 10000 1500
-F 0 "D2" H 9991 1716 50  0000 C CNN
-F 1 "LED" H 9991 1625 50  0000 C CNN
-F 2 "LEDs:LED_0805" H 10000 1500 50  0001 C CNN
-F 3 "~" H 10000 1500 50  0001 C CNN
-	1    10000 1500
-	1    0    0    -1
-$EndComp
-Wire Wire Line
-	10150 1500 10350 1500
+P 10050 2150
+F 0 "D2" H 10041 2366 50  0000 C CNN
+F 1 "LED" H 10041 2275 50  0000 C CNN
+F 2 "LEDs:LED_0805" H 10050 2150 50  0001 C CNN
+F 3 "~" H 10050 2150 50  0001 C CNN
+	1    10050 2150
+	-1   0    0    1
+$EndComp
+Wire Wire Line
+	10200 2150 10400 2150
 $Comp
 L Device:R_Small R5
 U 1 1 5E920474
-P 10450 1800
-F 0 "R5" V 10254 1800 50  0000 C CNN
-F 1 "300r" V 10345 1800 50  0000 C CNN
-F 2 "Resistor_SMD:R_0603_1608Metric_Pad1.05x0.95mm_HandSolder" H 10450 1800 50  0001 C CNN
-F 3 "~" H 10450 1800 50  0001 C CNN
-	1    10450 1800
+P 10450 950
+F 0 "R5" V 10254 950 50  0000 C CNN
+F 1 "300r" V 10345 950 50  0000 C CNN
+F 2 "Resistor_SMD:R_0603_1608Metric_Pad1.05x0.95mm_HandSolder" H 10450 950 50  0001 C CNN
+F 3 "~" H 10450 950 50  0001 C CNN
+	1    10450 950
 	0    1    1    0
 $EndComp
@@
 L Device:LED D3
 U 1 1 5E92047B
-P 10000 1800
-F 0 "D3" H 9991 2016 50  0000 C CNN
-F 1 "LED" H 9991 1925 50  0000 C CNN
-F 2 "LEDs:LED_0805" H 10000 1800 50  0001 C CNN
-F 3 "~" H 10000 1800 50  0001 C CNN
-	1    10000 1800
-	1    0    0    -1
-$EndComp
-Wire Wire Line
-	10150 1800 10350 1800
-Wire Wire Line
-	10550 1800 10800 1800
-Wire Wire Line
-	10800 1150 10800 1500
-Wire Wire Line
-	9850 1800 9550 1800
-Wire Wire Line
-	9550 1800 9550 2100
+P 10000 950
+F 0 "D3" H 9991 1166 50  0000 C CNN
+F 1 "LED" H 9991 1075 50  0000 C CNN
+F 2 "LEDs:LED_0805" H 10000 950 50  0001 C CNN
+F 3 "~" H 10000 950 50  0001 C CNN
+	1    10000 950
+	1    0    0    -1
+$EndComp
+Wire Wire Line
+	10150 950  10350 950
+Wire Wire Line
+	10550 950  10800 950
+Wire Wire Line
+	9850 950  9550 950
+Wire Wire Line
+	9550 950  9550 1250
 $Comp
 L power:GND #PWR0102
 U 1 1 5E920584
-P 9550 2100
-F 0 "#PWR0102" H 9550 1850 50  0001 C CNN
-F 1 "GND" H 9555 1927 50  0000 C CNN
-F 2 "" H 9550 2100 50  0001 C CNN
-F 3 "" H 9550 2100 50  0001 C CNN
-	1    9550 2100
-	1    0    0    -1
-$EndComp
-Wire Wire Line
-	9850 1500 9550 1500
-Wire Wire Line
-	9850 1150 9550 1150
+P 9550 1250
+F 0 "#PWR0102" H 9550 1000 50  0001 C CNN
+F 1 "GND" H 9555 1077 50  0000 C CNN
+F 2 "" H 9550 1250 50  0001 C CNN
+F 3 "" H 9550 1250 50  0001 C CNN
+	1    9550 1250
+	1    0    0    -1
+$EndComp
+Wire Wire Line
+	9900 2150 9600 2150
+Wire Wire Line
+	9900 1800 9600 1800
 Wire Wire Line
 	8050 1350 8500 1350
@@
 	1    0    0    -1
 $EndComp
-Text Label 9550 1150 2    50   ~ 0
+Text Label 9600 1800 2    50   ~ 0
 P3.0
-Text Label 9550 1500 2    50   ~ 0
+Text Label 9600 2150 2    50   ~ 0
 P3.1
-Text Notes 9750 1200 2    50   ~ 0
+Text Notes 9800 1850 2    50   ~ 0
 RX\n\n
-Text Notes 9750 1450 2    50   ~ 0
+Text Notes 9800 2100 2    50   ~ 0
 TX\n
-Text Notes 9750 1750 2    50   ~ 0
+Text Notes 9750 900  2    50   ~ 0
 POW\n
 Text Label 8500 1350 2    50   ~ 0
@@
 $EndComp
 Wire Wire Line
-	10550 1500 10800 1500
-Connection ~ 10800 1500
-Wire Wire Line
-	10800 1500 10800 1800
-$Comp
-L power:VCC #PWR?
+	10600 2150 10850 2150
+$Comp
+L power:VCC #PWR0121
 U 1 1 5EA08550
 P 10800 800
-F 0 "#PWR?" H 10800 650 50  0001 C CNN
+F 0 "#PWR0121" H 10800 650 50  0001 C CNN
 F 1 "VCC" H 10817 973 50  0000 C CNN
 F 2 "" H 10800 800 50  0001 C CNN
@@
 	1    0    0    -1
 $EndComp
+Wire Wire Line
+	10800 800  10800 950
+Wire Wire Line
+	10850 1800 10850 2150
+Wire Wire Line
+	10850 2150 10850 2500
+Connection ~ 10850 2150
+$Comp
+L power:GND #PWR0122
+U 1 1 5EA2494F
+P 10850 2500
+F 0 "#PWR0122" H 10850 2250 50  0001 C CNN
+F 1 "GND" H 10855 2327 50  0000 C CNN
+F 2 "" H 10850 2500 50  0001 C CNN
+F 3 "" H 10850 2500 50  0001 C CNN
+	1    10850 2500
+	1    0    0    -1
+$EndComp

Commit message: tied bootloader switch to gnd not vcc and silk fixes
Parts:
- removed R1: 10k, Resistor_SMD:R_0603_1608Metric_Pad1.05x0.95mm_HandSolder, symbol Device:R_Small
Connections:
- wire segments 119 -> 118
Changed lines of the file:
@@
 P3.7
-$Comp
-L Device:R_Small R1
-U 1 1 5E93B481
-P 800 1800
-F 0 "R1" H 741 1754 50  0000 R CNN
-F 1 "10k" H 741 1845 50  0000 R CNN
-F 2 "Resistor_SMD:R_0603_1608Metric_Pad1.05x0.95mm_HandSolder" H 800 1800 50  0001 C CNN
-F 3 "~" H 800 1800 50  0001 C CNN
-	1    800  1800
-	-1   0    0    1
-$EndComp
 $Comp
 L Device:C_Small C3
@@
 $EndComp
 Wire Wire Line
-	800  1900 800  2000
-Wire Wire Line
-	800  2000 1300 2000
-Wire Wire Line
-	800  1700 800  1350
-Wire Wire Line
 	1850 1800 1850 1650
 Wire Wire Line
@@
 Wire Wire Line
 	1850 2300 2650 2300
-$Comp
-L power:VCC #PWR0113
-U 1 1 5E9432E6
-P 800 1350
-F 0 "#PWR0113" H 800 1200 50  0001 C CNN
-F 1 "VCC" H 817 1523 50  0000 C CNN
-F 2 "" H 800 1350 50  0001 C CNN
-F 3 "" H 800 1350 50  0001 C CNN
-	1    800  1350
-	1    0    0    -1
-$EndComp
 $Comp
 L Device:R_Small R2
@@
 	1    0    0    -1
 $EndComp
+Wire Wire Line
+	850  2000 850  2350
+Wire Wire Line
+	850  2000 1300 2000
+$Comp
+L power:GND #PWR?
+U 1 1 5EB4598F
+P 850 2350
+F 0 "#PWR?" H 850 2100 50  0001 C CNN
+F 1 "GND" H 855 2177 50  0000 C CNN
+F 2 "" H 850 2350 50  0001 C CNN
+F 3 "" H 850 2350 50  0001 C CNN
+	1    850  2350
+	1    0    0    -1
+$EndComp

Commit message: checked and sent to porduction
Parts:
- removed JP1: SolderJumper_3_Bridged12, Jumper:SolderJumper-3_P1.3mm_Bridged2Bar12_RoundedPad1.0x1.5mm, symbol Jumper:SolderJumper_3_Bridged12
- removed R2: 10k, Resistor_SMD:R_0603_1608Metric_Pad1.05x0.95mm_HandSolder, symbol Device:R_Small
Connections:
- wire segments 118 -> 117
Changed lines of the file:
@@
 Text Label 5200 5200 2    50   ~ 0
 P1.4
-Text Label 2650 2300 2    50   ~ 0
-P1.5
 Text Label 5200 5500 2    50   ~ 0
 P1.6
@@
 Text Label 2650 1650 2    50   ~ 0
 P3.6
-$Comp
-L Jumper:SolderJumper_3_Bridged12 JP1
-U 1 1 5E93B8DD
-P 1850 2000
-F 0 "JP1" V 1804 2067 50  0000 L CNN
-F 1 "SolderJumper_3_Bridged12" V 1895 2067 50  0000 L CNN
-F 2 "Jumper:SolderJumper-3_P1.3mm_Bridged2Bar12_RoundedPad1.0x1.5mm" H 1850 2000 50  0001 C CNN
-F 3 "~" H 1850 2000 50  0001 C CNN
-	1    1850 2000
-	0    1    1    0
-$EndComp
-Wire Wire Line
-	1850 1800 1850 1650
 Wire Wire Line
 	1850 1650 2650 1650
-Wire Wire Line
-	1850 2200 1850 2300
-Wire Wire Line
-	1850 2300 2650 2300
-$Comp
-L Device:R_Small R2
-U 1 1 5E9433DF
-P 4050 1500
-F 0 "R2" H 3991 1454 50  0000 R CNN
-F 1 "10k" H 3991 1545 50  0000 R CNN
-F 2 "Resistor_SMD:R_0603_1608Metric_Pad1.05x0.95mm_HandSolder" H 4050 1500 50  0001 C CNN
-F 3 "~" H 4050 1500 50  0001 C CNN
-	1    4050 1500
-	-1   0    0    1
-$EndComp
-Wire Wire Line
-	4050 1600 4050 1850
 Wire Wire Line
 	4050 1850 4450 1850
@@
 	4450 1850 5100 1850
 Wire Wire Line
-	4050 1400 4050 1050
-Wire Wire Line
 	4050 1050 4450 1050
 Wire Wire Line
 	4450 1050 4450 1400
-Connection ~ 4050 1050
 Wire Wire Line
 	4050 1050 4050 850
@@
 L Switch:SW_Push SW2
 U 1 1 5E94BC64
-P 4050 2050
-F 0 "SW2" V 4096 2002 50  0000 R CNN
-F 1 "SW_Push" V 4005 2002 50  0000 R CNN
-F 2 "Button_Switch_SMD:SW_SPST_PTS810" H 4050 2250 50  0001 C CNN
-F 3 "" H 4050 2250 50  0001 C CNN
-	1    4050 2050
+P 4050 1400
+F 0 "SW2" V 4096 1352 50  0000 R CNN
+F 1 "SW_Push" V 4005 1352 50  0000 R CNN
+F 2 "Button_Switch_SMD:SW_SPST_PTS810" H 4050 1600 50  0001 C CNN
+F 3 "" H 4050 1600 50  0001 C CNN
+	1    4050 1400
 	0    -1   -1   0
 $EndComp
-Connection ~ 4050 1850
 Wire Wire Line
 	4050 2250 4050 2550
@@
 Wire Wire Line
 	7750 1950 7750 2150
-Text Notes 3850 2000 2    79   ~ 0
+Text Notes 3800 1400 2    79   ~ 0
 Reset\n
 Text Label 2550 2850 2    50   ~ 0
@@
 $EndComp
 Wire Wire Line
-	850  2000 850  2350
-Wire Wire Line
-	850  2000 1300 2000
-$Comp
-L power:GND #PWR?
-U 1 1 5EB4598F
-P 850 2350
-F 0 "#PWR?" H 850 2100 50  0001 C CNN
-F 1 "GND" H 855 2177 50  0000 C CNN
-F 2 "" H 850 2350 50  0001 C CNN
-F 3 "" H 850 2350 50  0001 C CNN
-	1    850  2350
-	1    0    0    -1
-$EndComp
+	4050 1050 4050 1200
+Connection ~ 4050 1050
+Wire Wire Line
+	4050 1600 4050 1850
+Wire Wire Line
+	800  1550 800  2000
+Wire Wire Line
+	800  2000 1300 2000
+Wire Wire Line
+	1700 2000 1850 2000
+Wire Wire Line
+	1850 1650 1850 2000
+$Comp
+L power:+3V3 #PWR?
+U 1 1 5EC0190F
+P 800 1550
+F 0 "#PWR?" H 800 1400 50  0001 C CNN
+F 1 "+3V3" H 815 1723 50  0000 C CNN
+F 2 "" H 800 1550 50  0001 C CNN
+F 3 "" H 800 1550 50  0001 C CNN
+	1    800  1550
+	1    0    0    -1
+$EndComp

Commit message: started updating schematic for version2
Parts:
- removed C4: 100nF, Capacitor_SMD:C_0603_1608Metric_Pad1.05x0.95mm_HandSolder, symbol Device:C_Small
- removed J3: USB_B_Micro, digikey-footprints:USB_Micro_B_Female_10118193-0001LF, symbol Connector:USB_B_Micro
- added C? (x2): 100nF, Capacitor_SMD:C_0603_1608Metric_Pad1.05x0.95mm_HandSolder, symbol Device:C_Small
- added D?: D_ALT, symbol Device:D_ALT
- added J?: USB_C_Receptacle, symbol Connector:USB_C_Receptacle
- added JP? (x2): Jumper, symbol Device:Jumper
- added Q?: CPH6337, symbol OnSemi:CPH6337
- added U?: MIC5504-3.3YM5, Package_TO_SOT_SMD:SOT-23-5, symbol Regulator_Linear:MIC5504-3.3YM5
Connections:
- net labels added: CC1, CC2, VBUS
- wire segments 117 -> 154
Other:
- note added: "Reverse Protection\n"

Commit message: Update CH552-USB-Devboard.sch
Parts:
- C4, C7: renamed from C?; value 100nF -> 1uF
- gave numbers to parts that had none: 6
Connections:
- wire segments 154 -> 157
Other:
- note added: "Prevents Reverse powering of VBUS"
Changed lines of the file:
@@
 	1850 1650 1850 2000
 $Comp
-L power:+3V3 #PWR?
+L power:+3V3 #PWR0101
 U 1 1 5EC0190F
 P 800 1550
-F 0 "#PWR?" H 800 1400 50  0001 C CNN
+F 0 "#PWR0101" H 800 1400 50  0001 C CNN
 F 1 "+3V3" H 815 1723 50  0000 C CNN
 F 2 "" H 800 1550 50  0001 C CNN
@@
 $EndComp
 $Comp
-L Regulator_Linear:MIC5504-3.3YM5 U?
+L Regulator_Linear:MIC5504-3.3YM5 U3
 U 1 1 5F0EED8D
 P 8450 2550
-F 0 "U?" H 8450 2917 50  0000 C CNN
+F 0 "U3" H 8450 2917 50  0000 C CNN
 F 1 "MIC5504-3.3YM5" H 8450 2826 50  0000 C CNN
 F 2 "Package_TO_SOT_SMD:SOT-23-5" H 8450 2150 50  0001 C CNN
@@
 $EndComp
 $Comp
-L Connector:USB_C_Receptacle J?
+L Connector:USB_C_Receptacle J3
 U 1 1 5F0EEE62
 P 5650 2150
-F 0 "J?" H 5755 3717 50  0000 C CNN
+F 0 "J3" H 5755 3717 50  0000 C CNN
 F 1 "USB_C_Receptacle" H 5755 3626 50  0000 C CNN
 F 2 "" H 5800 2150 50  0001 C CNN
@@
 Connection ~ 5750 4100
 $Comp
-L power:GND #PWR?
+L power:GND #PWR0103
 U 1 1 5F12C15E
 P 5750 4350
-F 0 "#PWR?" H 5750 4100 50  0001 C CNN
+F 0 "#PWR0103" H 5750 4100 50  0001 C CNN
 F 1 "GND" H 5755 4177 50  0000 C CNN
 F 2 "" H 5750 4350 50  0001 C CNN
@@
 	6750 950  6750 850
 $Comp
-L power:VBUS #PWR?
+L power:VBUS #PWR0104
 U 1 1 5F1419FC
 P 6750 700
-F 0 "#PWR?" H 6750 550 50  0001 C CNN
+F 0 "#PWR0104" H 6750 550 50  0001 C CNN
 F 1 "VBUS" H 6765 873 50  0000 C CNN
 F 2 "" H 6750 700 50  0001 C CNN
@@
 	1    0    0    -1
 $EndComp
-$Comp
-L Device:D_ALT D?
-U 1 1 5F141ABF
-P 10050 2950
-F 0 "D?" H 10050 3166 50  0000 C CNN
-F 1 "D_ALT" H 10050 3075 50  0000 C CNN
-F 2 "" H 10050 2950 50  0001 C CNN
-F 3 "~" H 10050 2950 50  0001 C CNN
-	1    10050 2950
-	1    0    0    -1
-$EndComp
 Wire Wire Line
 	10200 2950 10850 2950
@@
 	9600 2950 9600 2650
 $Comp
-L power:VCC #PWR?
+L power:VCC #PWR0113
 U 1 1 5F14D4F5
 P 9600 2650
-F 0 "#PWR?" H 9600 2500 50  0001 C CNN
+F 0 "#PWR0113" H 9600 2500 50  0001 C CNN
 F 1 "VCC" H 9617 2823 50  0000 C CNN
 F 2 "" H 9600 2650 50  0001 C CNN
@@
 $EndComp
 $Comp
-L power:GND #PWR?
+L power:GND #PWR0115
 U 1 1 5F14D56E
 P 10850 3150
-F 0 "#PWR?" H 10850 2900 50  0001 C CNN
+F 0 "#PWR0115" H 10850 2900 50  0001 C CNN
 F 1 "GND" H 10855 2977 50  0000 C CNN
 F 2 "" H 10850 3150 50  0001 C CNN
@@
 	9100 2150 9100 2450
 $Comp
-L power:+3V3 #PWR?
+L power:+3V3 #PWR0123
 U 1 1 5F17F9E8
 P 9100 2150
-F 0 "#PWR?" H 9100 2000 50  0001 C CNN
+F 0 "#PWR0123" H 9100 2000 50  0001 C CNN
 F 1 "+3V3" H 9115 2323 50  0000 C CNN
 F 2 "" H 9100 2150 50  0001 C CNN
@@
 $EndComp
 $Comp
-L power:VCC #PWR?
+L power:VCC #PWR0124
 U 1 1 5F17FAB9
 P 7800 2150
-F 0 "#PWR?" H 7800 2000 50  0001 C CNN
+F 0 "#PWR0124" H 7800 2000 50  0001 C CNN
 F 1 "VCC" H 7817 2323 50  0000 C CNN
 F 2 "" H 7800 2150 50  0001 C CNN
@@
 $EndComp
 $Comp
-L Device:C_Small C?
+L Device:C_Small C4
 U 1 1 5F17FBB6
 P 7500 2650
-F 0 "C?" H 7592 2696 50  0000 L CNN
-F 1 "100nF" H 7592 2605 50  0000 L CNN
+F 0 "C4" H 7592 2696 50  0000 L CNN
+F 1 "1uF" H 7592 2605 50  0000 L CNN
 F 2 "Capacitor_SMD:C_0603_1608Metric_Pad1.05x0.95mm_HandSolder" H 7500 2650 50  0001 C CNN
 F 3 "~" H 7500 2650 50  0001 C CNN
@@
 $EndComp
 $Comp
-L Device:C_Small C?
+L Device:C_Small C7
 U 1 1 5F17FC66
 P 9100 2650
-F 0 "C?" H 9192 2696 50  0000 L CNN
-F 1 "100nF" H 9192 2605 50  0000 L CNN
+F 0 "C7" H 9192 2696 50  0000 L CNN
+F 1 "1uF" H 9192 2605 50  0000 L CNN
 F 2 "Capacitor_SMD:C_0603_1608Metric_Pad1.05x0.95mm_HandSolder" H 9100 2650 50  0001 C CNN
 F 3 "~" H 9100 2650 50  0001 C CNN
@@
 	7500 2750 7500 3000
 $Comp
-L power:GND #PWR?
+L power:GND #PWR0125
 U 1 1 5F1936CC
 P 9100 3000
-F 0 "#PWR?" H 9100 2750 50  0001 C CNN
+F 0 "#PWR0125" H 9100 2750 50  0001 C CNN
 F 1 "GND" H 9105 2827 50  0000 C CNN
 F 2 "" H 9100 3000 50  0001 C CNN
@@
 $EndComp
 $Comp
-L power:GND #PWR?
+L power:GND #PWR0126
 U 1 1 5F19374F
 P 8450 3000
-F 0 "#PWR?" H 8450 2750 50  0001 C CNN
+F 0 "#PWR0126" H 8450 2750 50  0001 C CNN
 F 1 "GND" H 8455 2827 50  0000 C CNN
 F 2 "" H 8450 3000 50  0001 C CNN
@@
 $EndComp
 $Comp
-L power:GND #PWR?
+L power:GND #PWR0127
 U 1 1 5F19378A
 P 7500 3000
-F 0 "#PWR?" H 7500 2750 50  0001 C CNN
+F 0 "#PWR0127" H 7500 2750 50  0001 C CNN
 F 1 "GND" H 7505 2827 50  0000 C CNN
 F 2 "" H 7500 3000 50  0001 C CNN
@@
 Text Label 6700 1450 0    50   ~ 0
 CC2
-Text Label 3000 2800 0    50   ~ 0
-CC1
-Text Label 3000 2950 0    50   ~ 0
-CC2
-$Comp
-L Device:Jumper JP?
+$Comp
+L Device:Jumper JP1
 U 1 1 5F1A134B
 P 8250 1150
-F 0 "JP?" H 8250 1414 50  0000 C CNN
+F 0 "JP1" H 8250 1414 50  0000 C CNN
 F 1 "Jumper" H 8250 1323 50  0000 C CNN
 F 2 "" H 8250 1150 50  0001 C CNN
@@
 $EndComp
 $Comp
-L Device:Jumper JP?
+L Device:Jumper JP2
 U 1 1 5F1A13E3
 P 8250 1500
-F 0 "JP?" H 8250 1764 50  0000 C CNN
+F 0 "JP2" H 8250 1764 50  0000 C CNN
 F 1 "Jumper" H 8250 1673 50  0000 C CNN
 F 2 "" H 8250 1500 50  0001 C CNN
@@
 P1.5
 $Comp
-L OnSemi:CPH6337 Q?
+L OnSemi:CPH6337 Q1
 U 1 1 5F1BBBBE
 P 3650 3450
-F 0 "Q?" V 3900 3450 50  0000 C CNN
+F 0 "Q1" V 3900 3450 50  0000 C CNN
 F 1 "CPH6337" V 3991 3450 50  0000 C CNN
 F 2 "" H 3850 3550 50  0001 C CNN
@@
 Wire Wire Line
 	3450 3550 2850 3550
+Wire Wire Line
+	4350 3550 4350 3450
+Wire Wire Line
+	2850 3550 2850 3450
+$Comp
+L power:VBUS #PWR0128
+U 1 1 5F0F1905
+P 2850 3450
+F 0 "#PWR0128" H 2850 3300 50  0001 C CNN
+F 1 "VBUS" H 2865 3623 50  0000 C CNN
+F 2 "" H 2850 3450 50  0001 C CNN
+F 3 "" H 2850 3450 50  0001 C CNN
+	1    2850 3450
+	1    0    0    -1
+$EndComp
+$Comp
+L power:VCC #PWR0129
+U 1 1 5F0F19FA
+P 4350 3450
+F 0 "#PWR0129" H 4350 3300 50  0001 C CNN
+F 1 "VCC" H 4367 3623 50  0000 C CNN
+F 2 "" H 4350 3450 50  0001 C CNN
+F 3 "" H 4350 3450 50  0001 C CNN
+	1    4350 3450
+	1    0    0    -1
+$EndComp
+Text Notes 2950 3900 0    50   ~ 0
+Prevents Reverse powering of VBUS
+$Comp
+L Device:D_ALT D4
+U 1 1 5F141ABF
+P 10050 2950
+F 0 "D4" H 10050 3166 50  0000 C CNN
+F 1 "D_ALT" H 10050 3075 50  0000 C CNN
+F 2 "" H 10050 2950 50  0001 C CNN
+F 3 "~" H 10050 2950 50  0001 C CNN
+	1    10050 2950
+	1    0    0    -1
+$EndComp
+Wire Wire Line
+	3650 3250 3650 3000
+$Comp
+L power:VCC #PWR0130
+U 1 1 5F107E69
+P 3650 3000
+F 0 "#PWR0130" H 3650 2850 50  0001 C CNN
+F 1 "VCC" H 3667 3173 50  0000 C CNN
+F 2 "" H 3650 3000 50  0001 C CNN
+F 3 "" H 3650 3000 50  0001 C CNN
+	1    3650 3000
+	1    0    0    -1
+$EndComp
 $EndSCHEMATC
