File: CH552-USB-Devboard/_saved_CH552-USB-Devboard.sch (KiCad schematic (older format))
At the start: 26 parts, among them J1 Conn_01x11_Male, J2 Conn_01x11_Male, J3 USB_C_Receptacle, Q1 CPH6337, SW1 SW_Push, SW2 SW_Push, U1 CH552T, U2 CH552G, U3 MIC5504-3.3YM5, Y1 Crystal

Commit message: added V2 BOM
Parts:
- J3: symbol CH552-USB-Devboard-rescue:USB_C_Receptacle-Connector -> Connector:USB_C_Receptacle
- R3, R4: value 330r -> 1k
- R5: value 300r -> 1k
Changed lines of the file:
@@
 EESchema Schematic File Version 4
-EELAYER 30 0
+LIBS:CH552-USB-Devboard-cache
+EELAYER 26 0
 EELAYER END
 $Descr A4 11693 8268
@@
 P 10500 1800
 F 0 "R3" V 10304 1800 50  0000 C CNN
-F 1 "330r" V 10395 1800 50  0000 C CNN
+F 1 "1k" V 10395 1800 50  0000 C CNN
 F 2 "Resistor_SMD:R_0603_1608Metric_Pad1.05x0.95mm_HandSolder" H 10500 1800 50  0001 C CNN
 F 3 "~" H 10500 1800 50  0001 C CNN
@@
 P 10500 2150
 F 0 "R4" V 10304 2150 50  0000 C CNN
-F 1 "330r" V 10395 2150 50  0000 C CNN
+F 1 "1k" V 10395 2150 50  0000 C CNN
 F 2 "Resistor_SMD:R_0603_1608Metric_Pad1.05x0.95mm_HandSolder" H 10500 2150 50  0001 C CNN
 F 3 "~" H 10500 2150 50  0001 C CNN
@@
 P 10450 950
 F 0 "R5" V 10254 950 50  0000 C CNN
-F 1 "300r" V 10345 950 50  0000 C CNN
+F 1 "1k" V 10345 950 50  0000 C CNN
 F 2 "Resistor_SMD:R_0603_1608Metric_Pad1.05x0.95mm_HandSolder" H 10450 950 50  0001 C CNN
 F 3 "~" H 10450 950 50  0001 C CNN
@@
 $EndComp
 $Comp
-L CH552-USB-Devboard-rescue:USB_C_Receptacle-Connector J3
+L Connector:USB_C_Receptacle J3
 U 1 1 5F0EEE62
 P 5650 2150
